Commit message: Rename some files, using base which is compatible with open manipulator

File: turtlebot3_description/urdf/turtlebot3_waffle_for_open_manipulator.gazebo.xacro (robot description, xacro)
@@ -8,6 +8,6 @@
   </gazebo>
   <gazebo reference="wheel_left_link">
-    <mu1>0.1</mu1>
-    <mu2>0.1</mu2>
+    <mu1>10000</mu1>
+    <mu2>10000</mu2>
     <kp>500000.0</kp>
     <kd>10.0</kd>
@@ -18,6 +18,6 @@
   </gazebo>
   <gazebo reference="wheel_right_link">
-    <mu1>0.1</mu1>
-    <mu2>0.1</mu2>
+    <mu1>10000</mu1>
+    <mu2>10000</mu2>
     <kp>500000.0</kp>
     <kd>10.0</kd>
@@ -52,4 +52,5 @@
     <material>Gazebo/Grey</material>
   </gazebo>
+  <!-- Differential drive controller. -->
   <gazebo>
     <plugin name="turtlebot3_waffle_controller" filename="libgazebo_ros_diff_drive.so">
@@ -74,4 +75,5 @@
     </plugin>
   </gazebo>
+  <!-- IMU unit. -->
   <gazebo>
     <plugin name="imu_plugin" filename="libgazebo_ros_imu.so">
@@ -102,4 +104,5 @@
     </plugin>
   </gazebo>
+  <!-- Laser scan. -->
   <gazebo reference="base_scan">
     <material>Gazebo/FlatBlack</material>
@@ -134,5 +137,6 @@
     </sensor>
   </gazebo>
-  <gazebo reference="camera_rgb_frame">
+  <!-- Depth camera. -->
+  <gazebo reference="camera_depth_frame">
     <sensor type="depth" name="realsense_R200">
       <always_on>true</always_on>
@@ -176,21 +180,24 @@
       </plugin>
     </sensor>
+  </gazebo>
+  <!-- RGB camera. -->
+  <gazebo reference="camera_rgb_frame">
     <sensor type="camera" name="rgb_camera">
-      <always_on>true</always_on>
-      <visualize>$(arg camera_visual)</visualize>
-      <camera>
-          <horizontal_fov>1.3439</horizontal_fov>
-          <image>
-              <width>1280</width>
-              <height>720</height>
-              <format>R8G8B8</format>
-          </image>
-          <depth_camera></depth_camera>
-          <clip>
-              <near>0.03</near>
-              <far>100</far>
-          </clip>
-      </camera>
-    </sensor>
+    <always_on>true</always_on>
+    <visualize>$(arg camera_visual)</visualize>
+    <camera>
+        <horizontal_fov>1.3439</horizontal_fov>
+        <image>
+            <width>1280</width>
+            <height>720</height>
+            <format>R8G8B8</format>
+        </image>
+        <depth_camera></depth_camera>
+        <clip>
+            <near>0.03</near>
+            <far>100</far>
+        </clip>
+    </camera>
+  </sensor>
   </gazebo>
 </robot>

File: turtlebot3_description/urdf/turtlebot3_waffle_for_open_manipulator.urdf.xacro (robot description, xacro)
@@ -2,5 +2,5 @@
 <robot name="turtlebot3_waffle_for_open_manipulator" xmlns:xacro="http://ros.org/wiki/xacro">
   <xacro:include filename="$(find turtlebot3_description)/urdf/common_properties.xacro"/>
-  <xacro:include filename="$(find turtlebot3_description)/urdf/turtlebot3_waffle_pi_for_open_manipulator.gazebo.xacro"/>
+  <xacro:include filename="$(find turtlebot3_description)/urdf/turtlebot3_waffle_for_open_manipulator.gazebo.xacro"/>
   <xacro:property name="r200_cam_rgb_px" value="0.005"/>
   <xacro:property name="r200_cam_rgb_py" value="0.018"/>
@@ -145,5 +145,5 @@
     <parent link="base_link"/>
     <child link="base_scan"/>
-    <origin xyz="-0.024 0 0.122" rpy="0 0 0"/>
+    <origin xyz="-0.024 0 0.13" rpy="0 0 0"/>
   </joint>
   <link name="base_scan">
