Commit message: Added start scripts and removed unnecessary .world files

File: turtlebot3_description/urdf/turtlebot3_waffle_for_open_manipulator.urdf.xacro (robot description, xacro)
@@ -28,6 +28,5 @@
     </collision>
     <inertial>
-      <!-- <origin xyz="-0.064 0 0" rpy="0 0 0"/> -->
-      <origin xyz="-5.8190646e-02 3.8892103e-02 6.3998774e-02" rpy="0 0 0"/>
+      <origin xyz="-0.064 0 0.047" rpy="0 0 0"/>
       <mass value="2.7771056e+00"/>
       <!-- <mass value="1.7771056e+00"/> -->
@@ -35,7 +34,7 @@
                 <!-- iyy="4.8786869e-02" iyz="1.4954898e-05" -->
                 <!-- izz="3.9852748e-02" /> -->
-      <inertia ixx="1" ixy="0" ixz="0"
-                iyy="1" iyz="0"
-                izz="1" />
+      <inertia ixx="1e-3" ixy="0" ixz="0"
+                iyy="1e-3" iyz="0"
+                izz="1e-3" />
     </inertial>
   </link>
@@ -63,6 +62,6 @@
       <origin xyz="0 0 0" />
       <mass value="2.8498940e-02" />
-      <inertia ixx="1.1175580e-05" ixy="-4.2369783e-11" ixz="-5.9381719e-09"
-               iyy="1.1192413e-05" iyz="-1.4400107e-11"
+      <inertia ixx="1.1175580e-05" ixy="0" ixz="0"
+               iyy="1.1192413e-05" iyz="0"
                izz="2.0712558e-05" />
       </inertial>
@@ -91,6 +90,6 @@
       <origin xyz="0 0 0" />
       <mass value="2.8498940e-02" />
-      <inertia ixx="1.1175580e-05" ixy="-4.2369783e-11" ixz="-5.9381719e-09"
-               iyy="1.1192413e-05" iyz="-1.4400107e-11"
+      <inertia ixx="1.1175580e-05" ixy="0" ixz="0"
+               iyy="1.1192413e-05" iyz="0"
                izz="2.0712558e-05" />
       </inertial>
