Commit message: Make GUI plugin work in Gazebo; modified code for inertia

File: turtlebot3_description/urdf/turtlebot3_waffle.urdf.xacro (robot description, xacro)
@@ -27,10 +27,18 @@
       </geometry>
     </collision>
+    <!-- Original values. -->
+    <!-- <inertial> -->
+      <!-- <origin xyz="0 0 0" rpy="0 0 0"/> -->
+      <!-- <mass value="1.3729096e+00"/> -->
+      <!-- <inertia ixx="8.7002718e-03" ixy="-4.7576583e-05" ixz="1.1160499e-04" -->
+               <!-- iyy="8.6195418e-03" iyz="-3.5422299e-06" -->
+               <!-- izz="1.4612727e-02" /> -->
+    <!-- </inertial> -->
     <inertial>
       <origin xyz="0 0 0" rpy="0 0 0"/>
       <mass value="1.3729096e+00"/>
-      <inertia ixx="8.7002718e-03" ixy="-4.7576583e-05" ixz="1.1160499e-04"
-               iyy="8.6195418e-03" iyz="-3.5422299e-06"
-               izz="1.4612727e-02" />
+      <inertia ixx="1e-03" ixy="0" ixz="0"
+               iyy="1e-03" iyz="0"
+               izz="1e-03" />
     </inertial>
   </link>
